File: PCB/Power.kicad_sch (KiCad schematic)
At the start: 8 parts, among them Q101 FDN306P, U101 LM1117MP-3.3

Commit message: Made changes discussed in the design review
Parts:
- removed TP101: VCC, TestPoint:TestPoint_Pad_D1.5mm, symbol Connector:TestPoint
- removed TP102: 3.3v, TestPoint:TestPoint_Pad_D1.5mm, symbol Connector:TestPoint
Connections:
- net VIN renamed VBAT

Commit message: - Added missing inductor to make it work with 915 Mhz - Added digikey part number as a property - Reran jobset - Removed out of date BOM.xlsx - Attempted to use the config addon (didn't fully work)
Parts:
- C101: Digikey-PN (none) -> 311-1088-1-ND
- D101: Digikey-PN (none) -> 3147-B1931UD--05D000314U1930CT-ND
- Q101: Digikey-PN (none) -> 5399-FDN306PCT-ND
- R101, R102: Digikey-PN (none) -> RMCF0603FT1K00CT-ND
- U101: Digikey-PN (none) -> LM1117MP-3.3/NOPBCT-ND
Changed lines of the file:
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@@
 			)
 		)
-		(property "LCSC" ""
-			(at 63.5 55.88 0)
-			(hide yes)
-			(show_name no)
-			(do_not_autoplace no)
-			(effects
-				(font
-					(size 1.27 1.27)
-				)
-			)
-		)
-		(property "LCSC  Part #" ""
+		(property "Digikey-PN" "311-1088-1-ND"
 			(at 63.5 55.88 0)
 			(hide yes)
@@
 			)
 		)
-		(property "LCSC" ""
-			(at 194.31 62.23 0)
-			(hide yes)
-			(show_name no)
-			(do_not_autoplace no)
-			(effects
-				(font
-					(size 1.27 1.27)
-				)
-			)
-		)
-		(property "LCSC  Part #" ""
+		(property "Digikey-PN" "RMCF0603FT1K00CT-ND"
 			(at 194.31 62.23 0)
 			(hide yes)
@@
 			)
 		)
+		(property "Digikey-PN" "LM1117MP-3.3/NOPBCT-ND"
+			(at 50.8 49.53 0)
+			(hide yes)
+			(show_name no)
+			(do_not_autoplace no)
+			(effects
+				(font
+					(size 1.27 1.27)
+				)
+			)
+		)
 		(pin "1"
 		)
@@
 			)
 		)
+		(property "Digikey-PN" "5399-FDN306PCT-ND"
+			(at 194.31 50.8 90)
+			(hide yes)
+			(show_name no)
+			(do_not_autoplace no)
+			(effects
+				(font
+					(size 1.27 1.27)
+				)
+			)
+		)
 		(pin "2"
 		)
@@
 			)
 		)
-		(property "LCSC" ""
-			(at 106.68 59.69 0)
-			(hide yes)
-			(show_name no)
-			(do_not_autoplace no)
-			(effects
-				(font
-					(size 1.27 1.27)
-				)
-			)
-		)
-		(property "LCSC  Part #" ""
+		(property "Digikey-PN" "RMCF0603FT1K00CT-ND"
 			(at 106.68 59.69 0)
 			(hide yes)
@@
 			)
 		)
-		(property "LCSC" ""
+		(property "Digikey-PN" "3147-B1931UD--05D000314U1930CT-ND"
 			(at 106.68 46.99 90)
 			(hide yes)
-			(show_name no)
-			(do_not_autoplace no)
-			(effects
-				(font
-					(size 1.27 1.27)
-				)
-			)
-		)
-		(property "LCSC  Part #" ""
-			(at 106.68 46.99 90)
-			(hide yes)
