File: PCB/Radio.kicad_sch (KiCad schematic)
At the start: 29 parts, among them J501 Conn_Coaxial, U501 SX1262IMLTRT, U502 SKY13453-385LF, Y501 32 MHz

Commit message: - Added missing inductor to make it work with 915 Mhz - Added digikey part number as a property - Reran jobset - Removed out of date BOM.xlsx - Attempted to use the config addon (didn't fully work)
Parts:
- added L507: 0R, Inductor_SMD:L_0603_1608Metric_Pad1.05x0.95mm_HandSolder, symbol Device:L
- C501, C502, C503, C514, C515: Digikey-PN (none) -> 311-1088-1-ND
- C504, C512: Digikey-PN (none) -> 1276-1008-1-ND
- C505: Digikey-PN (none) -> 1276-1063-1-ND
- C506: Digikey-PN (none) -> 1276-6534-1-ND
- C507: Digikey-PN (none) -> 1276-6549-1-ND; Var(433MHz) (none) -> 3.3p; Var(915MHz) (none) -> 5.6; Var.Aspect (none) -> RadioFrequency
- C508: Digikey-PN (none) -> 1276-1792-1-ND; Var(433MHz) (none) -> 4.7p; Var(915MHz) (none) -> 1.5p; Var.Aspect (none) -> RadioFrequency
- C509: Digikey-PN (none) -> 399-C0603C109D4HACTUCT-ND; Var(433MHz) (none) -> 1p; Var(915MHz) (none) -> 0 -!; Var.Aspect (none) -> RadioFrequency
- C510: Digikey-PN (none) -> 1276-6549-1-ND; Var(433MHz) (none) -> 3.3p; Var(915MHz) (none) -> 0 -!; Var.Aspect (none) -> RadioFrequency
- C511: Digikey-PN (none) -> 1276-1089-1-ND; Var(433MHz) (none) -> 18p; Var(915MHz) (none) -> 5.6p; Var.Aspect (none) -> RadioFrequency
- C513: Digikey-PN (none) -> 1276-CL10C150JC81PNCCT-ND; Var(433MHz) (none) -> 15p; Var(915MHz) (none) -> 0 -!; Var.Aspect (none) -> RadioFrequency
- C516: Digikey-PN (none) -> 1276-1070-1-ND
- C517: now not fitted; now left out of the parts list
- C518: now not fitted
- J501: Digikey-PN (none) -> CON-SMA-EDGE-S-ND
- L501: Digikey-PN (none) -> 445-MLZ1608N150LT000CT-ND
- L502: Digikey-PN (none) -> 732-7447860168CT-ND; Var(433MHz) (none) -> 68n; Var(915MHz) (none) -> 68n; Var.Aspect (none) -> RadioFrequency
- L503: Digikey-PN (none) -> 478-LCCI0603J33NGTARCT-ND; Var(433MHz) (none) -> 33n; Var(915MHz) (none) -> 24n; Var.Aspect (none) -> RadioFrequency
- L504: Digikey-PN (none) -> 732-7447860039CT-ND; Var(433MHz) (none) -> 3.9n; Var(915MHz) (none) -> 6.5n; Var.Aspect (none) -> RadioFrequency
- L505: Digikey-PN (none) -> 732-7447860115CT-ND; Var(433MHz) (none) -> 15n; Var(915MHz) (none) -> 1.3n; Var.Aspect (none) -> RadioFrequency
- L506: Digikey-PN (none) -> 311-0.0LDCT-ND
- R501: Digikey-PN (none) -> 13-RT0603BRD07500RLCT-ND
- U501: Digikey-PN (none) -> SX1262IMLTRTCT-ND
- U502: Digikey-PN (none) -> 863-1602-1-ND
- Y501: Digikey-PN (none) -> 644-CS06654-32MCT-ND; private KLC_S4.1 -> KLC_S3.3
Connections:
- net RFO_0: now also L507.2; no longer C510.1, L502.2, L504.1
- net RFO_1: now also C510.1, L502.2, L504.1, L507.1; no longer C510.2, C511.1, L504.2, L505.2
- net RFO_2: now also C510.2, C511.1, L504.2, L505.2; no longer C512.2, L505.1
- net RFO_3: now also C512.2, L505.1; no longer C512.1, C513.1, U502.2 (RF1)
- new net RFO_4: C512.1, C513.1, U502.2 (RF1)
Other:
- moved on the sheet: C504, C506, C510, C511, L504, L505

Commit message: - Got the extension KiVar working to switch between a 433MHz and 915MHz radio - Added Digikey-PN's for the 915 MHz radio
Parts:
- C504: Var(433MHz) (none) -> 100p; Var(915MHz) (none) -> 100p; Var.Aspect (none) -> RadioFrequency
- C506: Var(433MHz) (none) -> 22n; Var(915MHz) (none) -> 22n; Var.Aspect (none) -> RadioFrequency
- C507: Digikey-PN.Var(433MHz) (none) -> 1276-6549-1-ND; Digikey-PN.Var(915MHz) (none) -> 399-C0603C569C5GACTUTR-ND; Var(915MHz) 5.6 -> 5.6p
- C508: Digikey-PN.Var(433MHz) (none) -> 1276-1792-1-ND; Digikey-PN.Var(915MHz) (none) -> 1292-HH18N1R5B500CTTR-ND
- C509: Digikey-PN.Var(433MHz) (none) -> 399-C0603C109D4HACTUCT-ND; Digikey-PN.Var(915MHz) (none) -> 0
- C510: Digikey-PN.Var(433MHz) (none) -> 1276-6549-1-ND; Digikey-PN.Var(915MHz) (none) -> 0
- C511: Digikey-PN.Var(433MHz) (none) -> 1276-1089-1-ND; Digikey-PN.Var(915MHz) (none) -> 399-C0603C569C5GACTUTR-ND
- C513: Digikey-PN.Var(433MHz) (none) -> 1276-CL10C150JC81PNCCT-ND; Digikey-PN.Var(915MHz) (none) -> 0
- L503: Digikey-PN.Var(433MHz) (none) -> 478-LCCI0603J33NGTARCT-ND; Digikey-PN.Var(915MHz) (none) -> 5262-HBWS1608-24NJTR-ND
- L504: Digikey-PN.Var(433MHz) (none) -> 732-7447860039CT-ND; Digikey-PN.Var(915MHz) (none) -> 490-LQW18AN6N5G80DTR-ND
- L505: Digikey-PN.Var(433MHz) (none) -> 732-7447860115CT-ND; Digikey-PN.Var(915MHz) (none) -> 535-11530-2-ND; Var(915MHz) 1.3n -> 1.2n
- L507: Digikey-PN.Var(433MHz) (none) -> 311-0.0LDCT-ND; Digikey-PN.Var(915MHz) (none) -> 490-LQW18AN6N5G80DTR-ND; KiLib_Generator (none) -> SMD_2terminal_chip_molded
- Y501: private KLC_S3.3 -> (none)
